Commit message: add front wheel

File: description/robot_core.xacro (robot description, xacro)
@@ -90,4 +90,50 @@
         </collision>
     </link>
+    <!-- LEFT FRONT WHEEL LINK -->
+    <joint name="left_front_wheel_joint" type="continuous">
+        <parent link="base_link"/>
+        <child link="left_front_wheel"/>
+        <origin xyz="0.29 0.09 0" rpy="-${pi/2} 0 0" />
+        <axis xyz="0 0 1"/>
+    </joint>
+    <link name="left_front_wheel">
+        <visual>
+            <geometry>
+                <cylinder radius="0.045" length="0.04"/>
+            </geometry>
+            <material name="black"/>
+        </visual>
+        <collision>
+            <geometry>
+                <cylinder radius="0.045" length="0.04"/>
+            </geometry>
+        </collision>
+        <xacro:inertial_cylinder mass="0.1" length="0.04" radius="0.045">
+            <origin xyz="0 0 0" rpy="0 0 0"/>
+        </xacro:inertial_cylinder>
+    </link>
+    <!-- right FRONT WHEEL LINK -->
+    <joint name="right_front_wheel_joint" type="continuous">
+        <parent link="base_link"/>
+        <child link="right_front_wheel"/>
+        <origin xyz=".29 -0.09 0" rpy="${pi/2} 0 0" />
+        <axis xyz="0 0 -1"/>
+    </joint>
+    <link name="right_front_wheel">
+        <visual>
+            <geometry>
+                <cylinder radius="0.045" length="0.04"/>
+            </geometry>
+            <material name="black"/>
+        </visual>
+        <collision>
+            <geometry>
+                <cylinder radius="0.045" length="0.04"/>
+            </geometry>
+        <xacro:inertial_cylinder mass="0.1" length="0.04" radius="0.045">
+            <origin xyz="0 0 0" rpy="0 0 0"/>
+        </xacro:inertial_cylinder>
+        </collision>
+    </link>
     <!-- CASTER WHEEL LINK -->
     <joint name="caster_wheel_joint" type="fixed">
