Commit message: fix Gazeboo and add wolrd

File: description/robot.urdf.xacro (robot description, xacro)
@@ -2,3 +2,4 @@
 <robot xmlns:xacro="http://www.ros.org/wiki/xacro"  name="robot">
     <xacro:include filename="robot_core.xacro" />
+    <xacro:include filename="gazebo_control.xacro" />
 </robot>

File: description/robot_core.xacro (robot description, xacro)
@@ -14,7 +14,4 @@
         <color rgba="0 0 0 1"/>
     </material>
-    <material name="red">
-        <color rgba="1 0 0 1"/>
-    </material>
     <!-- BASE LINK -->
     <link name="base_link">
@@ -24,35 +21,38 @@
         <parent link="base_link"/>
         <child link="chassis"/>
-        <origin xyz="0.05 0 0"/>
+        <origin xyz="-0.1 0 0"/>
     </joint>
     <link name="chassis">
         <visual>
-            <origin xyz="0.11 0 0.065"/>
+            <origin xyz="0.15 0 0.075"/>
             <geometry>
-                <box size="0.22 0.13 0.13"/>
+                <box size="0.3 0.3 0.15"/>
             </geometry>
             <material name="orange"/>
         </visual>
         <collision>
-            <origin xyz="0.11 0 0.065"/>
+            <origin xyz="0.15 0 0.075"/>
             <geometry>
-                <box size="0.22 0.13 0.13"/>
+                <box size="0.3 0.3 0.15"/>
             </geometry>
         </collision>
         <xacro:inertial_box mass="0.5" x="0.3" y="0.3" z="0.15">
-            <origin xyz="0.11 0 0.065" rpy="0 0 0"/>
+            <origin xyz="0.15 0 0.075" rpy="0 0 0"/>
         </xacro:inertial_box>
     </link>
-    <!-- LEFT BACK WHEEL LINK -->
-    <joint name="left_back_wheel_joint" type="continuous">
+    <gazebo reference="chassis">
+        <material>Gazebo/Orange</material>
+    </gazebo>
+    <!-- LEFT WHEEL LINK -->
+    <joint name="left_wheel_joint" type="continuous">
         <parent link="base_link"/>
-        <child link="left_back_wheel"/>
-        <origin xyz="0 0.09 0" rpy="-${pi/2} 0 0" />
+        <child link="left_wheel"/>
+        <origin xyz="0 0.175 0" rpy="-${pi/2} 0 0" />
         <axis xyz="0 0 1"/>
     </joint>
-    <link name="left_back_wheel">
+    <link name="left_wheel">
         <visual>
             <geometry>
-                <cylinder radius="0.045" length="0.04"/>
+                <cylinder radius="0.05" length="0.04"/>
             </geometry>
             <material name="black"/>
@@ -60,22 +60,25 @@
         <collision>
             <geometry>
-                <cylinder radius="0.045" length="0.04"/>
+                <cylinder radius="0.05" length="0.04"/>
             </geometry>
         </collision>
-        <xacro:inertial_cylinder mass="0.1" length="0.04" radius="0.045">
+        <xacro:inertial_cylinder mass="0.1" length="0.04" radius="0.05">
             <origin xyz="0 0 0" rpy="0 0 0"/>
         </xacro:inertial_cylinder>
     </link>
-    <!-- right BACK WHEEL LINK -->
-    <joint name="right_back_wheel_joint" type="continuous">
+    <gazebo reference="left_wheel">
+        <material>Gazebo/Black</material>
+    </gazebo>
+    <!-- RIGHT WHEEL LINK -->
+    <joint name="right_wheel_joint" type="continuous">
         <parent link="base_link"/>
-        <child link="right_back_wheel"/>
-        <origin xyz="0 -0.09 0" rpy="${pi/2} 0 0" />
+        <child link="right_wheel"/>
+        <origin xyz="0 -0.175 0" rpy="${pi/2} 0 0" />
         <axis xyz="0 0 -1"/>
     </joint>
-    <link name="right_back_wheel">
+    <link name="right_wheel">
         <visual>
             <geometry>
-                <cylinder radius="0.045" length="0.04"/>
+                <cylinder radius="0.05" length="0.04"/>
             </geometry>
             <material name="black"/>
@@ -83,16 +86,19 @@
         <collision>
             <geometry>
-                <cylinder radius="0.045" length="0.04"/>
+                <cylinder radius="0.05" length="0.04"/>
             </geometry>
-        <xacro:inertial_cylinder mass="0.1" length="0.04" radius="0.045">
+        </collision>
+        <xacro:inertial_cylinder mass="0.1" length="0.04" radius="0.05">
             <origin xyz="0 0 0" rpy="0 0 0"/>
         </xacro:inertial_cylinder>
-        </collision>
     </link>
-    <!-- LEFT FRONT WHEEL LINK -->
+    <gazebo reference="right_wheel">
+        <material>Gazebo/Black</material>
+    </gazebo>
+    <!-- LEFT front WHEEL LINK -->
     <joint name="left_front_wheel_joint" type="continuous">
         <parent link="base_link"/>
         <child link="left_front_wheel"/>
-        <origin xyz="0.29 0.09 0" rpy="-${pi/2} 0 0" />
+        <origin xyz="0.3 0.11 0" rpy="-${pi/2} 0 0" />
         <axis xyz="0 0 1"/>
     </joint>
@@ -100,22 +106,25 @@
         <visual>
             <geometry>
-                <cylinder radius="0.045" length="0.04"/>
+                <cylinder radius="0.05" length="0.04"/>
             </geometry>
-            <material name="black"/>
+            <material name="blue"/>
         </visual>
         <collision>
             <geometry>
-                <cylinder radius="0.045" length="0.04"/>
+                <cylinder radius="0.05" length="0.04"/>
             </geometry>
         </collision>
-        <xacro:inertial_cylinder mass="0.1" length="0.04" radius="0.045">
+        <xacro:inertial_cylinder mass="0.1" length="0.04" radius="0.05">
             <origin xyz="0 0 0" rpy="0 0 0"/>
         </xacro:inertial_cylinder>
     </link>
-    <!-- right FRONT WHEEL LINK -->
+    <gazebo reference="left_front_wheel">
+        <material>Gazebo/Black</material>
+    </gazebo>
+    <!-- RIGHT FRONT WHEEL LINK -->
     <joint name="right_front_wheel_joint" type="continuous">
         <parent link="base_link"/>
         <child link="right_front_wheel"/>
-        <origin xyz=".29 -0.09 0" rpy="${pi/2} 0 0" />
+        <origin xyz="0.3 -0.11 0" rpy="${pi/2} 0 0" />
         <axis xyz="0 0 -1"/>
     </joint>
@@ -123,22 +132,25 @@
         <visual>
             <geometry>
-                <cylinder radius="0.045" length="0.04"/>
+                <cylinder radius="0.05" length="0.04"/>
             </geometry>
-            <material name="black"/>
+            <material name="blue"/>
         </visual>
         <collision>
             <geometry>
-                <cylinder radius="0.045" length="0.04"/>
+                <cylinder radius="0.05" length="0.04"/>
             </geometry>
-        <xacro:inertial_cylinder mass="0.1" length="0.04" radius="0.045">
+        </collision>
+        <xacro:inertial_cylinder mass="0.1" length="0.04" radius="0.05">
             <origin xyz="0 0 0" rpy="0 0 0"/>
         </xacro:inertial_cylinder>
-        </collision>
     </link>
+    <gazebo reference="right_front_wheel">
+        <material>Gazebo/Black</material>
+    </gazebo>
     <!-- CASTER WHEEL LINK -->
     <joint name="caster_wheel_joint" type="fixed">
         <parent link="chassis"/>
         <child link="caster_wheel"/>
-        <origin xyz="0.055 0 0"/>
+        <origin xyz="0.24 0 0"/>
     </joint>
     <link name="caster_wheel">
@@ -147,14 +159,19 @@
                 <sphere radius="0.05"/>
             </geometry>
-            <material name="black"/>
+            <material name="orange"/>
         </visual>
         <collision>
             <geometry>
-                <sphere radius="0.045"/>
+                <sphere radius="0.05"/>
             </geometry>
         </collision>
-        <xacro:inertial_sphere mass="0.1" radius="0.045">
+        <xacro:inertial_sphere mass="0.1" radius="0.05">
             <origin xyz="0 0 0" rpy="0 0 0"/>
         </xacro:inertial_sphere>
     </link>
+    <gazebo reference="caster_wheel">
+        <material>Gazebo/Orange</material>
+        <mu1 value="0.001"/>
+        <mu2 value="0.001"/>
+    </gazebo>
 </robot>
